Commit message: Postęp

File: description/robot.urdf.xacro (robot description, xacro)
@@ -1,6 +1,6 @@
 <?xml version="1.0"?>
 <robot xmlns:xacro="http://www.ros.org/wiki/xacro" name="robot">
+    <xacro:arg name="sim_mode" default="false" />
     <xacro:include filename="robot_core.xacro"/>
-<!--<xacro:include filename="gazebo_control.xacro"/>   -->
     <xacro:include filename="$(find my_bot)/description/ros2_control.xacro" />
     <xacro:include filename="lidar.xacro"/>

File: description/ros2_control.xacro (robot description, xacro)
@@ -1,25 +1,88 @@
 <?xml version="1.0"?>
-<robot xmlns="http://www.ros.org">
-    <ros2_control name="GazeboSystem" type="system">
-        <hardware>
-            <plugin>gz_ros2_control/GazeboSimSystem</plugin>
-        </hardware>
-        <joint name="left_wheel_joint">
-            <command_interface name="velocity">
-                <param name="min">-10</param>
-                <param name="max">10</param>
-            </command_interface>
-            <state_interface name="velocity"/>
-            <state_interface name="position"/>
-        </joint>
-        <joint name="right_wheel_joint">
-            <command_interface name="velocity">
-                <param name="min">-10</param>
-                <param name="max">10</param>
-            </command_interface>
-            <state_interface name="velocity"/>
-            <state_interface name="position"/>
-        </joint>
-    </ros2_control>
+<robot xmlns:xacro="http://www.ros.org/wiki/xacro" xmlns="http://www.ros.org">
+    <xacro:unless value="$(arg sim_mode)">
+        <ros2_control name="RealRobot" type="system">
+            <hardware>
+                <plugin>diffdrive_arduino/DiffDriveArduino</plugin>
+                <param name="left_wheel_name">left_wheel_joint</param>
+                <param name="right_wheel_name">right_wheel_joint</param>
+                <param name="loop_rate">30</param>
+                <param name="device">/dev/ttyUSB0</param>
+                <param name="baud_rate">57600</param>
+                <param name="timeout">1000</param>
+                <param name="enc_counts_per_rev">1976</param>
+            </hardware>
+            <joint name="left_wheel_joint">
+                <command_interface name="velocity">
+                    <param name="min">-10</param>
+                    <param name="max">10</param>
+                </command_interface>
+                <state_interface name="velocity"/>
+                <state_interface name="position"/>
+            </joint>
+            <joint name="right_wheel_joint">
+                <command_interface name="velocity">
+                    <param name="min">-10</param>
+                    <param name="max">10</param>
+                </command_interface>
+                <state_interface name="velocity"/>
+                <state_interface name="position"/>
+            </jmjasic@RPi5:~/ros2_ws$ xacro ~/ros2_ws/src/my_bot/description/robot.urdf.xacro sim_mode:=false 2>&1 | head -50
+XML parsing error: unbound prefix: line 4, column 4
+when processing file: /home/mjasic/ros2_ws/install/my_bot/share/my_bot/description/ros2_control.xacro
+included from: /home/mjasic/ros2_ws/src/my_bot/description/robot.urdf.xacro
+Check that:
+ - Your XML is well-formed
+ - You have the xacro xmlns declaration: xmlns:xacro="http://www.ros.org/wiki/xacro"
+mjasic@RPi5:~/ros2_ws$ grep -n "include" ~/ros2_ws/src/my_bot/description/*.xacro
+/home/mjasic/ros2_ws/src/my_bot/description/robot_core.xacro:4:    <xacro:include filename="inertial_macros.xacro"/>
+/home/mjasic/ros2_ws/src/my_bot/description/robot.urdf.xacro:4:    <xacro:include filename="robot_core.xacro"/>
+/home/mjasic/ros2_ws/src/my_bot/description/robot.urdf.xacro:6:<!--<xacro:include filename="gazebo_control.xacro"/>   -->
+/home/mjasic/ros2_ws/src/my_bot/description/robot.urdf.xacro:7:    <xacro:include filename="$(find my_bot)/description/ros2_control.xacro" />
+/home/mjasic/ros2_ws/src/my_bot/description/robot.urdf.xacro:8:    <xacro:include filename="lidar.xacro"/>
+/home/mjasic/ros2_ws/src/my_bot/description/robot.urdf.xacro:9:    <xacro:include filename="camera.xacro"/>
+mjasic@RPi5:~/ros2_ws$ cd ~/ros2_ws
+rm -rf build/my_bot install/my_bot
+colcon build --symlink-install --packages-select my_bot
+source install/setup.bash
+xacro ~/ros2_ws/src/my_bot/description/robot.urdf.xacro sim_mode:=false | grep -A2 ros2_control
+[0.280s] WARNING:colcon.colcon_ros.prefix_path.ament:The path '/home/mjasic/ros2_ws/install/my_bot' in the environment variable AMENT_PREFIX_PATH doesn't exist
+[0.280s] WARNING:colcon.colcon_ros.prefix_path.catkin:The path '/home/mjasic/ros2_ws/install/my_bot' in the environment variable CMAKE_PREFIX_PATH doesn't exist
+Starting >>> my_bot
+Finished <<< my_bot [1.97s]
+Summary: 1 package finished [2.19s]
+XML parsing error: unbound prefix: line 4, column 4
+when processing file: /home/mjasic/ros2_ws/install/my_bot/share/my_bot/description/ros2_control.xacro
+included from: /home/mjasic/ros2_ws/src/my_bot/description/robot.urdf.xacro
+Check that:
+ - Your XML is well-formed
+ - You have the xacro xmlns declaration: xmlns:xacro="http://www.ros.org/wiki/xacro"
+mjasic@RPi5:~/ros2_ws$
+oint>
+        </ros2_control>
+    </xacro:unless>
+    <xacro:if value="$(arg sim_mode)">
+        <ros2_control name="GazeboSystem" type="system">
+            <hardware>
+                <plugin>gz_ros2_control/GazeboSimSystem</plugin>
+            </hardware>
+            <joint name="left_wheel_joint">
+                <command_interface name="velocity">
+                    <param name="min">-10</param>
+                    <param name="max">10</param>
+                </command_interface>
+                <state_interface name="velocity"/>
+                <state_interface name="position"/>
+            </joint>
+            <joint name="right_wheel_joint">
+                <command_interface name="velocity">
+                    <param name="min">-10</param>
+                    <param name="max">10</param>
+                </command_interface>
+                <state_interface name="velocity"/>
+                <state_interface name="position"/>
+            </joint>
+        </ros2_control>
+    </xacro:if>
     <gazebo>
         <plugin filename="libgz_ros2_control-system.so" name="gz_ros2_control::GazeboSimROS2ControlPlugin">
