Commit message: Tune Nav2 speed: RPP controller, rotation shim, real hardware limits

File: description/ros2_control.xacro (robot description, xacro)
@@ -15,14 +15,6 @@
             <joint name="left_wheel_joint">
                 <command_interface name="velocity">
-                    <param name="min">-10</param>
-                    <param name="max">10</param>
-                </command_interface>
-                <state_interface name="position"/>
-                <state_interface name="velocity"/>
-            </joint>
-            <joint name="right_wheel_joint">
-                <command_interface name="velocity">
-                    <param name="min">-10</param>
-                    <param name="max">10</param>
+                    <param name="min">-12</param>
+                    <param name="max">12</param>
                 </command_interface>
                 <state_interface name="position"/>
@@ -38,6 +30,6 @@
             <joint name="left_wheel_joint">
                 <command_interface name="velocity">
-                    <param name="min">-10</param>
-                    <param name="max">10</param>
+                    <param name="min">-12</param>
+                    <param name="max">12</param>
                 </command_interface>
                 <state_interface name="position"/>
@@ -46,6 +38,6 @@
             <joint name="right_wheel_joint">
                 <command_interface name="velocity">
-                    <param name="min">-10</param>
-                    <param name="max">10</param>
+                    <param name="min">-12</param>
+                    <param name="max">12</param>
                 </command_interface>
                 <state_interface name="position"/>
