Commit message: Initial commit

File: description/lidar.xacro (robot description, xacro)
@@ -47,5 +47,5 @@
             </ray>
             <always_on>true</always_on>
-            <visualize>false</visualize>
+            <visualize>true</visualize>
         </sensor>
     </gazebo>

File: description/robot_core.xacro (robot description, xacro)
@@ -24,4 +24,11 @@
         <origin xyz="-0.1 0 0"/>
     </joint>
+    <!-- Base footprint -->
+    <joint name="base_footprint_joint" type="fixed">
+        <parent link="base_link"/>
+        <child link="base_footprint"/>
+        <origin xyz="0 0 0" rpy="0 0 0"/>
+    </joint>
+    <link name="base_footprint"/>
     <link name="chassis">
         <visual>
@@ -49,5 +56,5 @@
         <parent link="base_link"/>
         <child link="left_wheel"/>
-        <origin xyz="0 0.175 0.05" rpy="-1.5708 0 0"/>
+        <origin xyz="0 0.125 0.0333" rpy="-1.5708 0 0"/>
         <axis xyz="0 0 1"/>
     </joint>
@@ -55,5 +62,5 @@
         <visual>
             <geometry>
-                <cylinder radius="0.05" length="0.04"/>
+                <cylinder radius="0.0333" length="0.04"/>
             </geometry>
             <material name="blue"/>
@@ -61,8 +68,8 @@
         <collision>
             <geometry>
-                <cylinder radius="0.05" length="0.04"/>
+                <cylinder radius="0.0333" length="0.04"/>
             </geometry>
         </collision>
-        <xacro:inertial_cylinder mass="0.1" length="0.04" radius="0.05">
+        <xacro:inertial_cylinder mass="0.1" length="0.04" radius="0.0333">
             <origin xyz="0 0 0" rpy="0 0 0"/>
         </xacro:inertial_cylinder>
@@ -75,5 +82,5 @@
         <parent link="base_link"/>
         <child link="right_wheel"/>
-        <origin xyz="0 -0.175 0.05" rpy="1.5708 0 0"/>
+        <origin xyz="0 -0.125 0.0333" rpy="1.5708 0 0"/>
         <axis xyz="0 0 -1"/>
     </joint>
@@ -81,5 +88,5 @@
         <visual>
             <geometry>
-                <cylinder radius="0.05" length="0.04"/>
+                <cylinder radius="0.0333" length="0.04"/>
             </geometry>
             <material name="blue"/>
@@ -87,8 +94,8 @@
         <collision>
             <geometry>
-                <cylinder radius="0.05" length="0.04"/>
+                <cylinder radius="0.0333" length="0.04"/>
             </geometry>
         </collision>
-        <xacro:inertial_cylinder mass="0.1" length="0.04" radius="0.05">
+        <xacro:inertial_cylinder mass="0.1" length="0.04" radius="0.0333">
             <origin xyz="0 0 0" rpy="0 0 0"/>
         </xacro:inertial_cylinder>
@@ -101,10 +108,10 @@
         <parent link="chassis"/>
         <child link="caster_wheel"/>
-        <origin xyz="0.24 0 0.05"/>
+        <origin xyz="0.24 0 0.0333"/>
     </joint>
     <link name="caster_wheel">
         <visual>
             <geometry>
-                <sphere radius="0.05"/>
+                <sphere radius="0.0333"/>
             </geometry>
             <material name="black"/>
@@ -112,8 +119,8 @@
         <collision>
             <geometry>
-                <sphere radius="0.05"/>
+                <sphere radius="0.0333"/>
             </geometry>
         </collision>
-        <xacro:inertial_sphere mass="0.1" radius="0.05">
+        <xacro:inertial_sphere mass="0.1" radius="0.0333">
             <origin xyz="0 0 0" rpy="0 0 0"/>
         </xacro:inertial_sphere>

File: description/ros2_control.xacro (robot description, xacro)
@@ -27,5 +27,8 @@
                 </command_interface>
                 <state_interface name="position"/>
+<<<<<<< HEAD
                 <state_interface name="velocity"/>
+=======
+>>>>>>> 6742c9e (Initial commit)
             </joint>
         </ros2_control>
