Commit message: Fix lidar 180 degree orientation offset

File: description/lidar.xacro (robot description, xacro)
@@ -21,5 +21,5 @@
         </collision>
         <xacro:inertial_cylinder mass="0.1" length="0.05" radius="0.04">
-            <origin xyz="0 0 0" rpy="0 0 0"/>
+            <origin xyz="0 0 0" rpy="0 0 3.14159"/>
         </xacro:inertial_cylinder>
     </link>

Commit message: Fix lidar 180 degree orientation (corrected joint origin, not inertial)

File: description/lidar.xacro (robot description, xacro)
@@ -4,5 +4,5 @@
         <parent link="chassis"/>
         <child link="laser_frame"/>
-        <origin xyz="0.1 0 0.22" rpy="0 0 0"/>
+        <origin xyz="0.1 0 0.22" rpy="0 0 3.14159"/>
     </joint>
     <link name="laser_frame">
@@ -21,5 +21,5 @@
         </collision>
         <xacro:inertial_cylinder mass="0.1" length="0.05" radius="0.04">
-            <origin xyz="0 0 0" rpy="0 0 3.14159"/>
+            <origin xyz="0 0 0" rpy="0 0 0"/>
         </xacro:inertial_cylinder>
     </link>
