Commit message: Add Nav2 configuration and fix wheel collision geometry

File: description/camera.xacro (robot description, xacro)
@@ -1,7 +1,4 @@
 <?xml version="1.0"?>
 <robot xmlns:xacro="http://www.ros.org/wiki/xacro">
-    <!-- ===================== -->
-    <!-- CAMERA MOUNT JOINT -->
-    <!-- ===================== -->
     <joint name="camera_joint" type="fixed">
         <parent link="chassis"/>
@@ -9,23 +6,12 @@
         <origin xyz="0.305 0 0.08" rpy="0 0 0"/>
     </joint>
-    <!-- ===================== -->
-    <!-- CAMERA LINK -->
-    <!-- ===================== -->
     <link name="camera_link">
         <visual>
             <geometry>
-                <box size="0.01 0.03 0.03"/>
+                <box size="0.010 0.03 0.03"/>
             </geometry>
-            <material name="red">
-                <color rgba="1 0 0 1"/>
-            </material>
+            <material name="red"/>
         </visual>
-        <collision>
-            <geometry>
-                <box size="0.01 0.03 0.03"/>
-            </geometry>
-        </collision>
     </link>
-    <!-- optical frame (ROS standard) -->
     <joint name="camera_optical_joint" type="fixed">
         <parent link="camera_link"/>
@@ -33,27 +19,25 @@
         <origin xyz="0 0 0" rpy="${-pi/2} 0 ${-pi/2}"/>
     </joint>
-    <link name="camera_link_optical"/>
-    <!-- ===================== -->
-    <!-- GAZEBO SENSOR -->
-    <!-- ===================== -->
+    <link name="camera_link_optical"></link>
     <gazebo reference="camera_link">
-        <!-- 🔥 Gazebo Sim sensor system (WAŻNE) -->
-        <plugin name="gz::sim::systems::Sensors"
-                filename="gz-sim-sensors-system"/>
+        <material>Gazebo/Red</material>
         <sensor name="camera" type="camera">
             <pose>0 0 0 0 0 0</pose>
-            <update_rate>30</update_rate>
+            <visualize>true</visualize>
+            <update_rate>10</update_rate>
+            <topic>camera/image_raw</topic>
             <camera>
                 <horizontal_fov>1.089</horizontal_fov>
                 <image>
+                    <format>R8G8B8</format>
                     <width>640</width>
                     <height>480</height>
-                    <format>R8G8B8</format>
                 </image>
                 <clip>
                     <near>0.05</near>
-                    <far>10.0</far>
+                    <far>8.0</far>
                 </clip>
             </camera>
+            <gz_frame_id>camera_link_optical</gz_frame_id>
         </sensor>
     </gazebo>

File: description/robot_core.xacro (robot description, xacro)
@@ -68,5 +68,5 @@
         <collision>
             <geometry>
-                <cylinder radius="0.0333" length="0.04"/>
+                <sphere radius="0.0333"/>
             </geometry>
         </collision>
@@ -94,5 +94,5 @@
         <collision>
             <geometry>
-                <cylinder radius="0.0333" length="0.04"/>
+                <sphere radius="0.0333"/>
             </geometry>
         </collision>

Commit message: Nowy model robota: wymiary, castery, maszt, lidar, Kinect, kamera

File: description/camera.xacro (robot description, xacro)
@@ -1,8 +1,9 @@
 <?xml version="1.0"?>
 <robot xmlns:xacro="http://www.ros.org/wiki/xacro">
+    <!-- ===== Raspberry Pi Camera 3 na przodzie podwozia (przod = x +0.265), wysokosc srodka podwozia ===== -->
     <joint name="camera_joint" type="fixed">
-        <parent link="chassis"/>
+        <parent link="base_link"/>
         <child link="camera_link"/>
-        <origin xyz="0.305 0 0.08" rpy="0 0 0"/>
+        <origin xyz="0.270 0 0.060" rpy="0 0 0"/>
     </joint>
     <link name="camera_link">
@@ -21,5 +22,4 @@
     <link name="camera_link_optical"></link>
     <gazebo reference="camera_link">
-        <material>Gazebo/Red</material>
         <sensor name="camera" type="camera">
             <pose>0 0 0 0 0 0</pose>
@@ -28,5 +28,6 @@
             <topic>camera/image_raw</topic>
             <camera>
-                <horizontal_fov>1.089</horizontal_fov>
+                <!-- Pi Camera 3 (standard) - ok. 66 stopni poziomo = 1.152 rad -->
+                <horizontal_fov>1.152</horizontal_fov>
                 <image>
                     <format>R8G8B8</format>
@@ -42,3 +43,38 @@
         </sensor>
     </gazebo>
+    <!-- ===== Kinect na maszcie, pod lidarem, przed masztem =====
+    Tylna scianka Kinecta przy przedniej scianie masztu (x = -0.180), srodek x = -0.145, z = 0.38. -->
+    <joint name="kinect_joint" type="fixed">
+        <parent link="base_link"/>
+        <child link="kinect_link"/>
+        <origin xyz="-0.145 0 0.380" rpy="0 0 0"/>
+    </joint>
+    <link name="kinect_link">
+        <visual>
+            <geometry>
+                <box size="0.070 0.280 0.065"/>
+            </geometry>
+            <material name="black"/>
+        </visual>
+        <collision>
+            <geometry>
+                <box size="0.070 0.280 0.065"/>
+            </geometry>
+        </collision>
+        <xacro:inertial_box mass="0.43" x="0.070" y="0.280" z="0.065">
+            <origin xyz="0 0 0" rpy="0 0 0"/>
+        </xacro:inertial_box>
+    </link>
+    <joint name="kinect_rgb_joint" type="fixed">
+        <parent link="kinect_link"/>
+        <child link="kinect_rgb"/>
+        <origin xyz="0.035 0 0" rpy="${-pi/2} 0 ${-pi/2}"/>
+    </joint>
+    <link name="kinect_rgb"></link>
+    <joint name="kinect_depth_joint" type="fixed">
+        <parent link="kinect_rgb"/>
+        <child link="kinect_depth"/>
+        <origin xyz="0.025 0 0" rpy="0 0 0"/>
+    </joint>
+    <link name="kinect_depth"></link>
 </robot>

File: description/lidar.xacro (robot description, xacro)
@@ -1,33 +1,38 @@
 <?xml version="1.0"?>
 <robot xmlns:xacro="http://www.ros.org/wiki/xacro">
+    <!--
+    RPLidar A1 na szczycie masztu. Ramka laser_frame = plaszczyzna skanowania,
+    0.450 m nad podlozem, 0.210 m za osia kol. Podstawa lidara jest na szczycie
+    masztu (0.415 m), wiec wizualnie walec ma srodek 0.0175 m ponizej ramki.
+    Obrot yaw = 3.14159 zostawiony jak w poprzedniej wersji (lidar montowany "tylem").
+    -->
     <joint name="laser_joint" type="fixed">
-        <parent link="chassis"/>
+        <parent link="base_link"/>
         <child link="laser_frame"/>
-        <origin xyz="0.1 0 0.22" rpy="0 0 3.14159"/>
+        <origin xyz="-0.210 0 0.450" rpy="0 0 3.14159"/>
     </joint>
     <link name="laser_frame">
         <visual>
+            <origin xyz="0 0 -0.0175" rpy="0 0 0"/>
             <geometry>
-                <cylinder radius="0.05" length="0.04"/>
+                <cylinder radius="0.036" length="0.035"/>
             </geometry>
-            <material name="red">
-                <color rgba="1 0 0 1"/>
-            </material>
+            <material name="red"/>
         </visual>
         <collision>
+            <origin xyz="0 0 -0.0175" rpy="0 0 0"/>
             <geometry>
-                <cylinder radius="0.04" length="0.05"/>
+                <cylinder radius="0.036" length="0.035"/>
             </geometry>
         </collision>
-        <xacro:inertial_cylinder mass="0.1" length="0.05" radius="0.04">
-            <origin xyz="0 0 0" rpy="0 0 0"/>
+        <xacro:inertial_cylinder mass="0.17" length="0.035" radius="0.036">
+            <origin xyz="0 0 -0.0175" rpy="0 0 0"/>
         </xacro:inertial_cylinder>
     </link>
     <gazebo reference="laser_frame">
-        <material>Gazebo/Red</material>
         <sensor name="laser" type="gpu_lidar">
             <gz_frame_id>laser_frame</gz_frame_id>
             <pose>0 0 0 0 0 0</pose>
-            <update_rate>10</update_rate>
+            <update_rate>5.5</update_rate>
             <topic>scan</topic>
             <ray>
@@ -41,8 +46,13 @@
                 </scan>
                 <range>
-                    <min>0.30</min>
+                    <min>0.15</min>
                     <max>12.0</max>
                     <resolution>0.01</resolution>
                 </range>
+                <noise>
+                    <type>gaussian</type>
+                    <mean>0.0</mean>
+                    <stddev>0.01</stddev>
+                </noise>
             </ray>
             <always_on>true</always_on>

File: description/robot_core.xacro (robot description, xacro)
@@ -1,4 +1,12 @@
 <?xml version="1.0"?>
 <robot xmlns:xacro="http://www.ros.org/wiki/xacro">
+    <!--
+    UKLAD ODNIESIENIA - base_link lezy na podlozu, dokladnie pod srodkiem osi kol napedowych.
+    x do przodu, y w lewo, z w gore. Wszystkie wymiary w metrach.
+    Wymiary robota (zmierzone)
+      kola 0.090 m srednicy, 0.022 m szerokosci, rozstaw 0.289 m
+      podwozie 0.530 x 0.326 x 0.080, przeswit 0.020
+      castery +/-0.180 m od osi, masa calego robota 6 kg
+    -->
     <xacro:include filename="inertial_macros.xacro"/>
     <material name="white">
@@ -17,11 +25,9 @@
         <color rgba="1 0 0 1"/>
     </material>
+    <material name="grey">
+        <color rgba="0.5 0.5 0.5 1"/>
+    </material>
     <!-- Base link -->
     <link name="base_link"/>
-    <joint name="chassis_joint" type="fixed">
-        <parent link="base_link"/>
-        <child link="chassis"/>
-        <origin xyz="-0.1 0 0"/>
-    </joint>
     <!-- Base footprint -->
     <joint name="base_footprint_joint" type="fixed">
@@ -31,30 +37,32 @@
     </joint>
     <link name="base_footprint"/>
+    <!-- Chassis - srodek podwozia lezy nad osia kol, 0.060 m nad podlozem (spod 0.020, gora 0.100) -->
+    <joint name="chassis_joint" type="fixed">
+        <parent link="base_link"/>
+        <child link="chassis"/>
+        <origin xyz="0 0 0.060"/>
+    </joint>
     <link name="chassis">
         <visual>
-            <origin xyz="0.15 0 0.125"/>
             <geometry>
-                <box size="0.3 0.3 0.15"/>
+                <box size="0.530 0.326 0.080"/>
             </geometry>
             <material name="white"/>
         </visual>
         <collision>
-            <origin xyz="0.15 0 0.125"/>
             <geometry>
-                <box size="0.3 0.3 0.15"/>
+                <box size="0.530 0.326 0.080"/>
             </geometry>
         </collision>
-        <xacro:inertial_box mass="0.5" x="0.3" y="0.3" z="0.15">
-            <origin xyz="0.15 0 0.125" rpy="0 0 0"/>
+        <!-- 4.85 kg - podwozie z akumulatorem, RPi, elektronika (6 kg calosc minus pozostale elementy) -->
+        <xacro:inertial_box mass="4.85" x="0.530" y="0.326" z="0.080">
+            <origin xyz="0 0 0" rpy="0 0 0"/>
         </xacro:inertial_box>
     </link>
-    <gazebo reference="chassis">
-        <material>Gazebo/White</material>
-    </gazebo>
     <!-- Left wheel -->
     <joint name="left_wheel_joint" type="continuous">
         <parent link="base_link"/>
         <child link="left_wheel"/>
-        <origin xyz="0 0.125 0.0333" rpy="-1.5708 0 0"/>
+        <origin xyz="0 0.1445 0.045" rpy="-1.5708 0 0"/>
         <axis xyz="0 0 1"/>
     </joint>
@@ -62,5 +70,5 @@
         <visual>
             <geometry>
-                <cylinder radius="0.0333" length="0.04"/>
+                <cylinder radius="0.045" length="0.022"/>
             </geometry>
             <material name="blue"/>
@@ -68,13 +76,14 @@
         <collision>
             <geometry>
-                <sphere radius="0.0333"/>
+                <sphere radius="0.045"/>
             </geometry>
         </collision>
-        <xacro:inertial_cylinder mass="0.1" length="0.04" radius="0.0333">
+        <xacro:inertial_cylinder mass="0.15" length="0.022" radius="0.045">
             <origin xyz="0 0 0" rpy="0 0 0"/>
         </xacro:inertial_cylinder>
     </link>
     <gazebo reference="left_wheel">
-        <material>Gazebo/Blue</material>
+        <mu1>1.0</mu1>
+        <mu2>1.0</mu2>
     </gazebo>
     <!-- Right wheel -->
@@ -82,5 +91,5 @@
         <parent link="base_link"/>
         <child link="right_wheel"/>
-        <origin xyz="0 -0.125 0.0333" rpy="1.5708 0 0"/>
+        <origin xyz="0 -0.1445 0.045" rpy="1.5708 0 0"/>
         <axis xyz="0 0 -1"/>
     </joint>
@@ -88,5 +97,5 @@
         <visual>
             <geometry>
-                <cylinder radius="0.0333" length="0.04"/>
+                <cylinder radius="0.045" length="0.022"/>
             </geometry>
             <material name="blue"/>
@@ -94,24 +103,30 @@
         <collision>
             <geometry>
-                <sphere radius="0.0333"/>
+                <sphere radius="0.045"/>
             </geometry>
         </collision>
-        <xacro:inertial_cylinder mass="0.1" length="0.04" radius="0.0333">
+        <xacro:inertial_cylinder mass="0.15" length="0.022" radius="0.045">
             <origin xyz="0 0 0" rpy="0 0 0"/>
         </xacro:inertial_cylinder>
     </link>
     <gazebo reference="right_wheel">
-        <material>Gazebo/Blue</material>
+        <mu1>1.0</mu1>
+        <mu2>1.0</mu2>
     </gazebo>
-    <!-- Caster wheel -->
-    <joint name="caster_wheel_joint" type="fixed">
-        <parent link="chassis"/>
-        <child link="caster_wheel"/>
-        <origin xyz="0.24 0 0.0333"/>
+    <!--
+    Castery (przedni i tylny) - kulki o promieniu 0.020 m.
+    Srodek kulki jest 0.5 mm powyzej "idealnego" kontaktu z podlozem, wiec
+    robot opiera sie na kolach napedowych (maja lepszy kontakt), a castery
+    tylko podtrzymuja go przy przechyle. Tarcie praktycznie zerowe.
+    -->
+    <joint name="front_caster_joint" type="fixed">
+        <parent link="base_link"/>
+        <child link="front_caster"/>
+        <origin xyz="0.180 0 0.0205"/>
     </joint>
-    <link name="caster_wheel">
+    <link name="front_caster">
         <visual>
             <geometry>
-                <sphere radius="0.0333"/>
+                <sphere radius="0.020"/>
             </geometry>
             <material name="black"/>
@@ -119,15 +134,65 @@
         <collision>
             <geometry>
-                <sphere radius="0.0333"/>
+                <sphere radius="0.020"/>
             </geometry>
         </collision>
-        <xacro:inertial_sphere mass="0.1" radius="0.0333">
+        <xacro:inertial_sphere mass="0.05" radius="0.020">
             <origin xyz="0 0 0" rpy="0 0 0"/>
         </xacro:inertial_sphere>
     </link>
-    <gazebo reference="caster_wheel">
-        <material>Gazebo/Black</material>
-        <mu1 value="0.001"/>
-        <mu2 value="0.001"/>
+    <gazebo reference="front_caster">
+        <mu1>0.001</mu1>
+        <mu2>0.001</mu2>
     </gazebo>
+    <joint name="rear_caster_joint" type="fixed">
+        <parent link="base_link"/>
+        <child link="rear_caster"/>
+        <origin xyz="-0.180 0 0.0205"/>
+    </joint>
+    <link name="rear_caster">
+        <visual>
+            <geometry>
+                <sphere radius="0.020"/>
+            </geometry>
+            <material name="black"/>
+        </visual>
+        <collision>
+            <geometry>
+                <sphere radius="0.020"/>
+            </geometry>
+        </collision>
+        <xacro:inertial_sphere mass="0.05" radius="0.020">
+            <origin xyz="0 0 0" rpy="0 0 0"/>
+        </xacro:inertial_sphere>
+    </link>
+    <gazebo reference="rear_caster">
+        <mu1>0.001</mu1>
+        <mu2>0.001</mu2>
+    </gazebo>
+    <!--
+    Maszt na tyle robota - 60 mm (x) x 40 mm (y), dlugosc 0.360 m.
+    Dol 0.055 m (schowany w podwoziu), gora 0.415 m. Srodek x = -0.210.
+    Na szczycie stoi lidar, nizej Kinect.
+    -->
+    <joint name="mast_joint" type="fixed">
+        <parent link="base_link"/>
+        <child link="mast"/>
+        <origin xyz="-0.210 0 0.235"/>
+    </joint>
+    <link name="mast">
+        <visual>
+            <geometry>
+                <box size="0.060 0.040 0.360"/>
+            </geometry>
+            <material name="grey"/>
+        </visual>
+        <collision>
+            <geometry>
+                <box size="0.060 0.040 0.360"/>
+            </geometry>
+        </collision>
+        <xacro:inertial_box mass="0.15" x="0.060" y="0.040" z="0.360">
+            <origin xyz="0 0 0" rpy="0 0 0"/>
+        </xacro:inertial_box>
+    </link>
 </robot>
